Commit message: tring out

File: urdf/udacity_bot.xacro (robot description, xacro)
@@ -1,3 +1,3 @@
-<?xml version='1.0'?>
+<?xml version="1.0"?>
 <robot name="udacity_bot" xmlns:xacro="http://www.ros.org/wiki/xacro">
   <xacro:include filename="$(find udacity_bot)/urdf/udacity_bot.gazebo" />
@@ -8,5 +8,5 @@
     <child link="chassis" />
   </joint>
-  <link name='chassis'>
+  <link name="chassis">
     <pose>0 0 0.1 0 0 0</pose>
     <inertial>
@@ -19,5 +19,5 @@
       />
     </inertial>
-    <collision name='collision'>
+    <collision name="collision">
       <origin xyz="0 0 0" rpy=" 0 0 0"/>
       <geometry>
@@ -25,15 +25,14 @@
       </geometry>
     </collision>
-    <visual name='chassis_visual'>
+    <visual name="chassis_visual">
       <origin xyz="0 0 0" rpy=" 0 0 0"/>
       <geometry>
         <box size=".4 .2 .1"/>
       </geometry>
-      <material name="red"/>
     </visual>
-    <collision name='back_caster_collision'>
+    <collision name="back_caster_collision">
       <origin xyz="-0.15 0 -0.05" rpy=" 0 0 0"/>
       <geometry>
-        <sphere radius="0.05"/>
+        <sphere radius="0.048"/>
       </geometry>
       <surface>
@@ -48,5 +47,5 @@
       </surface>
     </collision>
-    <visual name='back_caster_visual'>
+    <visual name="back_caster_visual">
       <origin xyz="-0.15 0 -0.05" rpy=" 0 0 0"/>
       <geometry>
@@ -54,8 +53,8 @@
       </geometry>
     </visual>
-    <collision name='front_caster_collision'>
+    <collision name="front_caster_collision">
       <origin xyz="0.15 0 -0.05" rpy=" 0 0 0"/>
       <geometry>
-        <sphere radius="0.05"/>
+        <sphere radius="0.048"/>
       </geometry>
       <surface>
@@ -70,5 +69,5 @@
       </surface>
     </collision>
-    <visual name='front_caster_visual'>
+    <visual name="front_caster_visual">
       <origin xyz="0.15 0 -0.05" rpy=" 0 0 0"/>
       <geometry>
@@ -77,9 +76,8 @@
     </visual>
   </link>
-  <!-- wheels -->
   <link name="left_wheel">
     <inertial>
       <mass value="5.0"/>
-      <origin xyz="0 0 0" rpy=" 0 1.5707 1.5707"/>
+      <origin xyz="0.0 0 0" rpy=" 0 0 0"/>
       <inertia
           ixx="0.1" ixy="0" ixz="0"
@@ -88,113 +86,111 @@
       />
     </inertial>
-    <collision name="collision">
-      <origin xyz="0 0 0" rpy=" 0 1.5707 1.5707"/>
+    <collision>
+      <origin xyz="0 0 0" rpy="1.5707 0 0"/>
       <geometry>
-        <cylinder radius="0.1" length="0.05" />
+        <cylinder radius=".1" length="0.05"/>
       </geometry>
     </collision>
-    <visual name="visual">
-      <origin xyz="0 0 0" rpy="0 1.5707 1.5707"/>
+    <visual>
+      <origin xyz="0 0 0" rpy="1.5707 0 0"/>
       <geometry>
-        <cylinder radius="0.1" length="0.05" />
+        <cylinder radius="0.1" length="0.05"/>
       </geometry>
     </visual>
-   </link>
-   <joint type="continuous" name="left_wheel_hinge">
-     <origin xyz="0 0.15 0" rpy="0 0 0"/>
-     <child link="left_wheel"/>
-     <parent link="chassis"/>
-     <axis xyz="0 1 0" rpy="0 0 0"/>
-     <limit effort="10000" velocity="1000"/>
-     <joint_properties damping="1.0" friction="1.0"/>
-   </joint>
-   <link name="right_wheel">
-     <inertial>
-       <mass value="5.0"/>
-       <origin xyz="0 0 0" rpy="0 1.5707 1.5707"/>
-       <inertia
+  </link>
+  <joint name="left_wheel_hinge" type="continuous">
+    <origin xyz="0.0 0.13 0" rpy="0 0 0"/>
+    <child link="left_wheel"/>
+    <parent link="chassis" />
+    <axis xyz="0 1 0" rpy="0 0 0" />
+    <limit effort="10000" velocity="1000" />
+    <joint_properties damping="1.0" friction="1.0" />
+  </joint>
+  <link name="right_wheel">
+    <inertial>
+      <mass value="5.0"/>
+      <origin xyz="0.0 0 0" rpy=" 0 0 0"/>
+      <inertia
           ixx="0.1" ixy="0" ixz="0"
           iyy="0.1" iyz="0"
           izz="0.1"
-	  />
-     </inertial>
-     <collision name="collision">
-       <origin xyz="0 0 0" rpy="0 1.5707 1.5707"/>
-       <geometry>
-         <cylinder radius="0.1" length="0.05" />
-       </geometry>
-     </collision>
-     <visual name="visual">
-       <origin xyz="0 0 0" rpy="0 1.5707 1.5707"/>
-       <geometry>
-         <cylinder radius="0.1" length="0.05" />
-       </geometry>
-     </visual>
-   </link>
-   <joint type="continuous" name="right_wheel_hinge">
-     <origin xyz="0 -0.15 0" rpy="0 0 0"/>
-     <child link="right_wheel"/>
-     <parent link="chassis"/>
-     <axis xyz="0 1 0" rpy="0 0 0"/>
-     <limit effort="10000" velocity="1000"/>
-     <joint_properties damping="1.0" friction="1.0"/>
-   </joint>
-   <!-- camera -->
-   <link name="camera">
-     <inertial>
-       <mass value="0.1"/>
-       <origin xyz="0 0 0" rpy="0 0 0"/>
-       <inertia
+      />
+    </inertial>
+    <collision>
+      <origin xyz="0 0 0" rpy="1.5707 0 0"/>
+      <geometry>
+        <cylinder radius=".1" length="0.05"/>
+      </geometry>
+    </collision>
+    <visual>
+      <origin xyz="0 0 0" rpy="1.5707 0 0"/>
+      <geometry>
+        <cylinder radius="0.1" length="0.05"/>
+      </geometry>
+    </visual>
+  </link>
+  <joint name="right_wheel_hinge" type="continuous">
+    <origin xyz="0.0 -0.13 0" rpy="0 0 0"/>
+    <child link="right_wheel"/>
+    <parent link="chassis" />
+    <axis xyz="0 1 0" rpy="0 0 0" />
+    <limit effort="10000" velocity="1000" />
+    <joint_properties damping="1.0" friction="1.0" />
+  </joint>
+  <joint name="camera_joint" type="fixed">
+    <origin xyz="0.2 0 0" rpy="0 0 0" />
+    <child link="camera" />
+    <parent link="chassis" />
+  </joint>
+  <link name="camera">
+    <inertial>
+      <mass value="0.1"/>
+      <origin xyz="0.0 0 0" rpy=" 0 0 0"/>
+      <inertia
           ixx="1e-6" ixy="0" ixz="0"
           iyy="1e-6" iyz="0"
           izz="1e-6"
-	  />
-       </inertial>
-       <collision name="collision">
-	 <origin xyz="0 0 0" rpy="0 0 0"/>
-	 <geometry>
-           <box size="0.05 0.05 0.05" />
-	 </geometry>
-       </collision>
-       <visual name="visual">
-	 <origin xyz="0 0 0" rpy="0 0 0"/>
-	 <geometry>
-           <box size="0.05 0.05 0.05" />
-	 </geometry>
-       </visual>
-   </link>
-   <joint type="fixed" name="camera_joint">
-     <origin xyz="0.2 0 0" rpy="0 0 0"/>
-     <child link="camera"/>
-     <parent link="chassis"/>
-   </joint>
-   <!-- lasor -->
-   <link name="hokuyo">
-     <inertial>
-       <mass value="0.1"/>
-       <origin xyz="0 0 0" rpy="0 0 0"/>
-       <inertia
-           ixx="1e-6" ixy="0" ixz="0"
-           iyy="1e-6" iyz="0"
-           izz="1e-6"
-	   />
-     </inertial>
-     <collision name="collision">
-       <origin xyz="0 0 0" rpy="0 0 0"/>
-       <geometry>
-         <box size="0.1 0.1 0.1" />
-       </geometry>
-     </collision>
-     <visual name="visual">
-       <origin xyz="0 0 0" rpy="0 0 0"/>
-       <geometry>
-         <mesh filename="package://udacity_bot/meshes/hokuyo.dae"/>
-       </geometry>
-     </visual>
-   </link>
-   <joint type="fixed" name="hokuyo_joint">
-     <origin xyz="0.15 0 0.1" rpy="0 0 0"/>
-     <child link="hokuyo"/>
-     <parent link="chassis"/>
-   </joint>
+      />
+    </inertial>
+    <collision>
+      <origin xyz="0 0 0" rpy=" 0 0 0"/>
+      <geometry>
+        <box size="0.05 0.05 0.05" />
+      </geometry>
+    </collision>
+    <visual>
+      <origin xyz="0 0 0" rpy=" 0 0 0"/>
+      <geometry>
+        <box size="0.05 0.05 0.05" />
+      </geometry>
+    </visual>
+  </link>
+  <joint name="hokuyo_joint" type="fixed">
+    <origin xyz="0.15 0 .1" rpy="0 0 0" />
+    <child link="hokuyo" />
+    <parent link="chassis" />
+  </joint>
+  <link name="hokuyo">
+    <inertial>
+      <mass value="0.1"/>
+      <origin xyz="0.0 0 0" rpy=" 0 0 0"/>
+      <inertia
+          ixx="1e-6" ixy="0" ixz="0"
+          iyy="1e-6" iyz="0"
+          izz="1e-6"
+      />
+    </inertial>
+    <collision>
+      <origin xyz="0 0 0" rpy="0 0 0"/>
+      <geometry>
+        <box size="0.1 0.1 0.1" />
+      </geometry>
+    </collision>
+    <visual>
+      <origin xyz="0 0 0" rpy="0 0 0"/>
+      <geometry>
+        <mesh filename="package://udacity_bot/meshes/hokuyo.dae" />
+      </geometry>
+    </visual>
+  </link>
 </robot>
